Commit message: update joint limits of urdf

File: urdf/amph.urdf (robot description, URDF)
Before this commit: robot amph, 17 links, 16 joints
Joints:
- joint Front_Left_Calf_joint: limit lower=-2.36 upper=0.79 effort=3.5 velocity=12 -> lower=-0.76 upper=2.36 effort=3.5 velocity=12
- joint Front_Left_Side_joint: limit lower=-0.52 upper=2.36 effort=3.5 velocity=12 -> lower=-2.36 upper=0.36 effort=3.5 velocity=12
- joint Front_Left_Thigh_joint: limit lower=-1.31 upper=1.31 effort=3.5 velocity=12 -> lower=-0.24 upper=1.31 effort=3.5 velocity=12
- joint Front_Right_Calf_joint: limit lower=-2.36 upper=0.79 effort=3.5 velocity=12 -> lower=-0.76 upper=2.36 effort=3.5 velocity=12
- joint Front_Right_Side_joint: limit lower=-2.36 upper=0.52 effort=3.5 velocity=12 -> lower=-0.36 upper=2.36 effort=3.5 velocity=12
- joint Front_Right_Thigh_joint: limit lower=-1.31 upper=1.31 effort=3.5 velocity=12 -> lower=-0.24 upper=1.31 effort=3.5 velocity=12
- joint Hind_Left_Calf_joint: limit lower=-2.36 upper=0.79 effort=3.5 velocity=12 -> lower=-0.76 upper=2.36 effort=3.5 velocity=12
- joint Hind_Left_Side_joint: limit lower=-0.52 upper=2.36 effort=3.5 velocity=12 -> lower=-0.36 upper=2.36 effort=3.5 velocity=12
- joint Hind_Left_Thigh_joint: limit lower=-1.31 upper=1.31 effort=3.5 velocity=12 -> lower=-0.24 upper=1.31 effort=3.5 velocity=12
- joint Hind_Right_Calf_joint: limit lower=-2.36 upper=0.79 effort=3.5 velocity=12 -> lower=-0.76 upper=2.36 effort=3.5 velocity=12
- joint Hind_Right_Side_joint: limit lower=-2.36 upper=0.52 effort=3.5 velocity=12 -> lower=-2.36 upper=0.36 effort=3.5 velocity=12
- joint Hind_Right_Thigh_joint: limit lower=-1.31 upper=1.31 effort=3.5 velocity=12 -> lower=-0.24 upper=1.31 effort=3.5 velocity=12
