Commit message: updates for body2

File: src/BODY2/urdf/BODY2.urdf (robot description, URDF)
Before this commit: robot BODY2, 25 links, 24 joints
Joints:
- joint Joint_BL1.1: origin xyz=-0.169151121513308 1.05843685412489 0.0640784613687492 rpy=1.5707963267949 -0.512211698143984 3.14159265358979 -> xyz=-0.0478568957987064 0.0502209715158126 0.0280761803936512 rpy=1.5707963267949 -0.512211698143984 0
- joint Joint_BL1.3: origin xyz=-0.0516119955246449 -0.00634051342585286 0.00300000000000021 rpy=0 0 0.91218357233305 -> xyz=-0.0516119955246449 -0.00634051342585283 0.00300000000000019 rpy=0 0 0.91218357233305
- joint Joint_BL2.1: origin xyz=-0.169151121513308 1.05993685412489 0.0360784613687492 rpy=1.5707963267949 0.336518268628592 -3.14159265358979 -> xyz=-0.0478568957987064 0.0487209715158128 7.61803936512387e-05 rpy=1.5707963267949 0.336518268628592 0
- joint Joint_BL2.3: origin xyz=0.049186953187325 0.0168713842148242 0 rpy=3.14159265358979 0 -1.67526464076333 -> xyz=0.049186953187325 0.0168713842148243 0 rpy=3.14159265358979 0 -1.67526464076333
- joint Joint_BR1.1: origin xyz=-0.169151121513308 1.15323685412489 0.0640784613687492 rpy=-1.5707963267949 -0.0578319161345941 3.14159265358979 -> xyz=-0.0478568957987064 -0.0445790284841874 0.0280761803936512 rpy=-1.5707963267949 -0.0578319161345941 0
- joint Joint_BR1.3: origin xyz=-0.051998029858748 0.000452695454739773 -0.00299999999999965 rpy=3.14159265358979 0 1.18094495136328 -> xyz=-0.051998029858748 0.000452695454739766 -0.00299999999999966 rpy=3.14159265358979 0 1.18094495136328
- joint Joint_BR2.1: origin xyz=-0.169151121513308 1.15323685412489 0.0360784613687492 rpy=-1.5707963267949 0.633858478635347 -3.14159265358979 -> xyz=-0.0478568957987064 -0.0445790284841874 7.61803936512387e-05 rpy=-1.5707963267949 0.633858478635347 0
- joint Joint_BR2.2: origin xyz=0.0299839903651189 -0.00097995504929356 -0.00329999999999973 rpy=0 0 -1.36396393396151 -> xyz=0.0299839903651189 -0.000979955049293556 -0.00329999999999972 rpy=0 0 -1.36396393396151
- joint Joint_BR2.3: origin xyz=-0.0518752774435282 0.0035993876242094 0.00299999999999975 rpy=3.14159265358979 0 1.36396393163113 -> xyz=-0.0518752774435282 0.00359938762420936 0.00299999999999974 rpy=3.14159265358979 0 1.36396393163113
- joint Joint_FL1.1: origin xyz=-0.308551121513308 1.05843685412489 0.0634784613687493 rpy=1.5707963267949 -0.0599910783746507 3.14159265358979 -> xyz=0.0915431042012935 0.0502209715158126 0.0274761803936513 rpy=1.5707963267949 -0.0599910783746507 0
- joint Joint_FL2.1: origin xyz=-0.308551121513308 1.05993685412489 0.0354784613687492 rpy=1.5707963267949 0.648496084693685 -3.14159265358979 -> xyz=0.0915431042012935 0.0487209715158128 -0.000523819606348758 rpy=1.5707963267949 0.648496084693685 0
- joint Joint_FL2.3: origin xyz=-0.051941819594197 0.00245912951712825 0 rpy=3.14159265358979 0 1.40056735852985 -> xyz=-0.0519418195941969 0.00245912951712825 0 rpy=3.14159265358979 0 1.40056735852985
- joint Joint_FR1.1: origin xyz=-0.308551121513308 1.15323685412489 0.0634784613687492 rpy=-1.5707963267949 -0.439226196697785 3.14159265358979 -> xyz=0.0915431042012936 -0.0445790284841874 0.0274761803936512 rpy=-1.5707963267949 -0.439226196697785 0
- joint Joint_FR1.2: origin xyz=0.0332346028261404 0.0109754784213317 -0.00479999999999955 rpy=0 0 1.49528079844306 -> xyz=0.0332346028261404 0.0109754784213317 -0.00479999999999954 rpy=0 0 1.49528079844306
- joint Joint_FR1.3: origin xyz=0.0512870600596529 0.00858122288813052 -0.00300000000000054 rpy=3.14159265358979 0 -1.9934298266756 -> xyz=0.0512870600596529 0.00858122288813053 -0.00300000000000054 rpy=3.14159265358979 0 -1.99342982667561
- joint Joint_FR2.1: origin xyz=-0.308551121513308 1.15323685412489 0.0354784613687492 rpy=-1.5707963267949 0.332932854178985 -3.14159265358979 -> xyz=0.0915431042012936 -0.0445790284841874 -0.000523819606348758 rpy=-1.5707963267949 0.332932854178986 0
- joint Joint_FR2.2: origin xyz=0.0289270491339261 0.00795146729797108 -0.0032999999999997 rpy=0 0 1.87128457541191 -> xyz=0.0289270491339261 0.00795146729797107 -0.00329999999999969 rpy=0 0 1.87128457541191
- joint Joint_FR2.3: origin xyz=0.0515056747457824 0.00715300535723657 0.00299999999999992 rpy=3.14159265358979 0 -1.87128457420229 -> xyz=0.0515056747457824 0.00715300535723653 0.00299999999999995 rpy=3.14159265358979 0 -1.87128457420228

Commit message: Spell BODY2's joint names with underscores instead of dots

File: src/BODY2/urdf/BODY2.urdf (robot description, URDF)
Before this commit: robot BODY2, 25 links, 24 joints
Joints:
- removed joint Joint_BL1.1
- removed joint Joint_BL1.2
- removed joint Joint_BL1.3
- removed joint Joint_BL2.1
- removed joint Joint_BL2.2
- removed joint Joint_BL2.3
- removed joint Joint_BR1.1
- removed joint Joint_BR1.2
- removed joint Joint_BR1.3
- removed joint Joint_BR2.1
- removed joint Joint_BR2.2
- removed joint Joint_BR2.3
- removed joint Joint_FL1.1
- removed joint Joint_FL1.2
- removed joint Joint_FL1.3
- removed joint Joint_FL2.1
- removed joint Joint_FL2.2
- removed joint Joint_FL2.3
- removed joint Joint_FR1.1
- removed joint Joint_FR1.2
- removed joint Joint_FR1.3
- removed joint Joint_FR2.1
- removed joint Joint_FR2.2
- removed joint Joint_FR2.3
- added joint Joint_BL1_1: type continuous, parent base_link, child Link_BL1.1, origin xyz=-0.0478568957987064 0.0502209715158126 0.0280761803936512 rpy=1.5707963267949 -0.512211698143984 0, axis 0 0 -1
- added joint Joint_BL1_2: type continuous, parent Link_BL1.1, child Link_BL1.2, origin xyz=0.0323457839693413 -0.0133697500892816 0 rpy=3.14159265358979 0 1.52978162195089, axis 0 0 1
- added joint Joint_BL1_3: type continuous, parent Link_BL1.2, child Link_BL1.3, origin xyz=-0.0516119955246449 -0.00634051342585276 0.00300000000000019 rpy=0 0 0.91218357233305, axis 0 0 1
- added joint Joint_BL2_1: type continuous, parent base_link, child Link_BL2.1, origin xyz=-0.0478568957987064 0.0487209715158128 7.61803936512387e-05 rpy=1.5707963267949 0.336518268628592 0, axis 0 0 -1
- added joint Joint_BL2_2: type continuous, parent Link_BL2.1, child Link_BL2.2, origin xyz=0.0289553723718933 -0.00784770102498905 0 rpy=3.14159265358979 0 -1.67526463585188, axis 0 0 1
- added joint Joint_BL2_3: type continuous, parent Link_BL2.2, child Link_BL2.3, origin xyz=0.049186953187325 0.0168713842148243 0 rpy=3.14159265358979 0 -1.67526464076333, axis 0 0 -1
- added joint Joint_BR1_1: type continuous, parent base_link, child Link_BR1.1, origin xyz=-0.0478568957987064 -0.0445790284841874 0.0280761803936512 rpy=-1.5707963267949 -0.0578319161345941 0, axis 0 0 -1
- added joint Joint_BR1_2: type continuous, parent Link_BR1.1, child Link_BR1.2, origin xyz=0.0349318189962401 -0.00218356265169693 -0.00479999999999959 rpy=0 0 -1.85321849201773, axis 0 0 1
- added joint Joint_BR1_3: type continuous, parent Link_BR1.2, child Link_BR1.3, origin xyz=-0.051998029858748 0.000452695454739773 -0.00299999999999966 rpy=3.14159265358979 0 1.18094495136328, axis 0 0 1
- added joint Joint_BR2_1: type continuous, parent base_link, child Link_BR2.1, origin xyz=-0.0478568957987064 -0.0445790284841874 7.61803936512387e-05 rpy=-1.5707963267949 0.633858478635348 0, axis 0 0 -1
- added joint Joint_BR2_2: type continuous, parent Link_BR2.1, child Link_BR2.2, origin xyz=0.0299839903651189 -0.000979955049293556 -0.00329999999999972 rpy=0 0 -1.36396393396151, axis 0 0 1
- added joint Joint_BR2_3: type continuous, parent Link_BR2.2, child Link_BR2.3, origin xyz=-0.0518752774435282 0.00359938762420931 0.00299999999999974 rpy=3.14159265358979 0 1.36396393163114, axis 0 0 1
- added joint Joint_FL1_1: type continuous, parent base_link, child Link_FL1.1, origin xyz=0.0915431042012935 0.0502209715158126 0.0274761803936513 rpy=1.5707963267949 -0.0599910783746507 0, axis 0 0 -1
- added joint Joint_FL1_2: type continuous, parent Link_FL1.1, child Link_FL1.2, origin xyz=0.0349364524941426 0.00210813417164982 0 rpy=3.14159265358979 0 1.83862774064259, axis 0 0 1
- added joint Joint_FL1_3: type continuous, parent Link_FL1.2, child Link_FL1.3, origin xyz=-0.0519883841796289 0.00109906138814747 0.00300000000000067 rpy=0 0 1.14654754518106, axis 0 0 1
- added joint Joint_FL2_1: type continuous, parent base_link, child Link_FL2.1, origin xyz=0.0915431042012935 0.0487209715158128 -0.000523819606348758 rpy=1.5707963267949 0.648496084693685 0, axis 0 0 -1
- added joint Joint_FL2_2: type continuous, parent Link_FL2.1, child Link_FL2.2, origin xyz=0.0299664342355442 0.00141872819801235 0 rpy=3.14159265358979 0 1.40056735852986, axis 0 0 1
- added joint Joint_FL2_3: type continuous, parent Link_FL2.2, child Link_FL2.3, origin xyz=-0.0519418195941969 0.00245912951712827 0 rpy=3.14159265358979 0 1.40056735852985, axis 0 0 -1
- added joint Joint_FR1_1: type continuous, parent base_link, child Link_FR1.1, origin xyz=0.0915431042012936 -0.0445790284841874 0.0274761803936512 rpy=-1.5707963267949 -0.439226196697785 0, axis 0 0 -1
- added joint Joint_FR1_2: type continuous, parent Link_FR1.1, child Link_FR1.2, origin xyz=0.0332346028261404 0.0109754784213317 -0.00479999999999954 rpy=0 0 1.49528079844306, axis 0 0 1
- added joint Joint_FR1_3: type continuous, parent Link_FR1.2, child Link_FR1.3, origin xyz=0.0512870600596529 0.00858122288813051 -0.00300000000000054 rpy=3.14159265358979 0 -1.99342982667561, axis 0 0 1
- added joint Joint_FR2_1: type continuous, parent base_link, child Link_FR2.1, origin xyz=0.0915431042012936 -0.0445790284841874 -0.000523819606348758 rpy=-1.5707963267949 0.332932854178986 0, axis 0 0 -1
- added joint Joint_FR2_2: type continuous, parent Link_FR2.1, child Link_FR2.2, origin xyz=0.0289270491339261 0.00795146729797108 -0.00329999999999969 rpy=0 0 1.87128457541191, axis 0 0 1
- added joint Joint_FR2_3: type continuous, parent Link_FR2.2, child Link_FR2.3, origin xyz=0.0515056747457824 0.00715300535723654 0.00299999999999995 rpy=3.14159265358979 0 -1.87128457420228, axis 0 0 1

Commit message: reduce jittering

File: src/BODY2/urdf/BODY2.urdf (robot description, URDF)
Before this commit: robot BODY2, 25 links, 24 joints
Links:
- link Link_BL1.1: mass 0.000223268078494629 -> 0.000900840261026578
- link Link_BL1.2: mass 0.000248010258828361 -> 0.000998814620637674
- link Link_BL2.1: mass 0.000240765805490465 -> 0.000972195105099795
- link Link_BR1.1: mass 0.000223268078494628 -> 0.000900840318089747
- link Link_BR1.2: mass 0.000248010258828361 -> 0.000998814653989497
- link Link_BR2.1: mass 0.000240765805490464 -> 0.000972195094897943
- link Link_FL1.1: mass 0.000223268078494629 -> 0.000900840181157897
- link Link_FL1.2: mass 0.00024801025882836 -> 0.000998814658375445
- link Link_FL2.1: mass 0.000240765805490465 -> 0.00097219515514233
- link Link_FR1.1: mass 0.000223268078494628 -> 0.000900840346021255
- link Link_FR1.2: mass 0.00024801025882836 -> 0.00099881458875752
- link Link_FR2.1: mass 0.000240765805490464 -> 0.000972195065668047
Joints:
- joint Joint_BL1_1: limit (none) -> effort=3.5 velocity=12
- joint Joint_BL1_2: limit (none) -> effort=3.5 velocity=12
- joint Joint_BL1_3: limit (none) -> effort=3.5 velocity=12
- joint Joint_BL2_1: limit (none) -> effort=3.5 velocity=12
- joint Joint_BL2_2: limit (none) -> effort=3.5 velocity=12
- joint Joint_BL2_3: limit (none) -> effort=3.5 velocity=12
- joint Joint_BR1_1: limit (none) -> effort=3.5 velocity=12
- joint Joint_BR1_2: limit (none) -> effort=3.5 velocity=12
- joint Joint_BR1_3: limit (none) -> effort=3.5 velocity=12
- joint Joint_BR2_1: limit (none) -> effort=3.5 velocity=12
- joint Joint_BR2_2: limit (none) -> effort=3.5 velocity=12
- joint Joint_BR2_3: limit (none) -> effort=3.5 velocity=12
- joint Joint_FL1_1: limit (none) -> effort=3.5 velocity=12
- joint Joint_FL1_2: limit (none) -> effort=3.5 velocity=12
- joint Joint_FL1_3: limit (none) -> effort=3.5 velocity=12
- joint Joint_FL2_1: limit (none) -> effort=3.5 velocity=12
- joint Joint_FL2_2: limit (none) -> effort=3.5 velocity=12
- joint Joint_FL2_3: limit (none) -> effort=3.5 velocity=12
- joint Joint_FR1_1: limit (none) -> effort=3.5 velocity=12
- joint Joint_FR1_2: limit (none) -> effort=3.5 velocity=12
- joint Joint_FR1_3: limit (none) -> effort=3.5 velocity=12
- joint Joint_FR2_1: limit (none) -> effort=3.5 velocity=12
- joint Joint_FR2_2: limit (none) -> effort=3.5 velocity=12
- joint Joint_FR2_3: limit (none) -> effort=3.5 velocity=12
